Commit message: 4wheeler 'URDF

File: urdf/fourwheeler.urdf (robot description, URDF)
Before this commit: robot fourwheeler, 1 links, 0 joints
Links:
- added link front_left_wheel; visual cylinder length=0.05 radius=0.1
- added link front_right_wheel; visual cylinder length=0.05 radius=0.1
- added link hood; visual box size=0.530 0.420 0.005
- added link lidar; visual cylinder length=0.08 radius=0.05
- added link rear_left_wheel; visual cylinder length=0.05 radius=0.1
- added link rear_right_wheel; visual cylinder length=0.05 radius=0.1
Joints:
- added joint front_left_wheel_to_base: type continuous, parent base_link, child front_left_wheel, origin xyz=0.1075 0.1851 -0.05 rpy=1.57 0 0, axis 0 0 1
- added joint front_right_wheel_to_base: type continuous, parent base_link, child front_right_wheel, origin xyz=0.1075 -0.1851 -0.05 rpy=1.57 0 0, axis 0 0 1
- added joint hood_to_base: type fixed, parent base_link, child hood, origin xyz=0 0 0.0725
- added joint lidar_to_hood: type continuous, parent hood, child lidar, origin xyz=0.15 0 0.04 rpy=0 0 0, axis 0 0 1
- added joint rear_left_wheel_to_base: type continuous, parent base_link, child rear_left_wheel, origin xyz=-0.1075 0.1851 -0.05 rpy=1.57 0 0, axis 0 0 1
- added joint rear_right_wheel_to_base: type continuous, parent base_link, child rear_right_wheel, origin xyz=-0.1075 -0.1851 -0.05 rpy=1.57 0 0, axis 0 0 1
