Commit message: 4wheeler parametrized

File: urdf/fourwheeler.urdf.xacro (robot description, xacro)
@@ -1,12 +1,15 @@
 <?xml version="1.0"?>
 <robot name="fourwheeler" xmlns:xacro="http://www.ros.org/wiki/xacro">
-    <xacro:property name="base_width" value="0.52"/>
-    <xacro:property name="wheel_width" value="0.05"/>
-    <xacro:property name="wheel_radius" value="0.1"/>
+    <xacro:property name="base_width" value="0.32"/> <!-- 0.32 -->
+    <xacro:property name="base_length" value="0.83"/> <!-- 0.43 -->
+    <xacro:property name="base_height" value="0.14"/> <!-- 0.14 -->
+    <xacro:property name="wheel_width" value="0.05"/> <!-- 0.05 -->
+    <xacro:property name="lowrider" value="0.01"/> <!-- 0 -->
+    <xacro:property name="wheel_radius" value="0.1"/> <!-- 0.1 -->
     <xacro:property name="half_track" value="${base_width/2 + wheel_width/2}"/>
     <link name="base_link">
         <visual>
             <geometry>
-            <box size="0.430 ${base_width} 0.140" />
+            <box size="${base_length} ${base_width} ${base_height}" />
             </geometry>
             <material name="blue">
@@ -29,5 +32,5 @@
             <parent link="base_link" />
             <child link="${wheel_name}" />
-            <origin xyz="${reflect_x * 0.1075} ${reflect_y * half_track} -0.05" rpy="1.57 0 0" />
+            <origin xyz="${reflect_x * (base_length/2 - wheel_radius)} ${reflect_y * half_track} ${lowrider-(base_height/2 - 0.02)}" rpy="1.57 0 0" />
             <axis xyz="0 0 1" />
         </joint>
@@ -40,5 +43,5 @@
         <visual>
             <geometry>
-            <box size="0.530 0.420 0.005" />
+            <box size="${base_length + 0.1} ${base_width} 0.005" />
             </geometry>
             <material name="yellow">
@@ -65,5 +68,5 @@
         <parent link="hood" />
         <child link="lidar" />
-        <origin xyz="0.15 0 0.04" rpy="0 0 0" />
+        <origin xyz="${base_length/2 - 0.065} 0 0.04" rpy="0 0 0" />
         <axis xyz="0 0 1" />
     </joint>

Commit message: 4wheeler drivable

File: urdf/fourwheeler.urdf.xacro (robot description, xacro)
@@ -1,11 +1,22 @@
 <?xml version="1.0"?>
 <robot name="fourwheeler" xmlns:xacro="http://www.ros.org/wiki/xacro">
+    <!-- constants; original values are in comments -->
     <xacro:property name="base_width" value="0.32"/> <!-- 0.32 -->
-    <xacro:property name="base_length" value="0.83"/> <!-- 0.43 -->
+    <xacro:property name="base_length" value="0.43"/> <!-- 0.43 -->
     <xacro:property name="base_height" value="0.14"/> <!-- 0.14 -->
     <xacro:property name="wheel_width" value="0.05"/> <!-- 0.05 -->
-    <xacro:property name="lowrider" value="0.01"/> <!-- 0 -->
+    <xacro:property name="lowrider" value="0"/> <!-- 0 -->
     <xacro:property name="wheel_radius" value="0.1"/> <!-- 0.1 -->
+    <!-- calculated parameters -->
     <xacro:property name="half_track" value="${base_width/2 + wheel_width/2}"/>
+    <xacro:property name="wheel_axis_z" value="${lowrider-(base_height/2 - 0.02)}"/>
+    <!-- model itself -->
+    <!-- invisible point at "floor" for driving model -->
+    <link name="base_footprint"></link>
+    <joint name="base_to_base_footprint" type="fixed">
+        <parent link="base_footprint" />
+        <child link="base_link" />
+        <origin xyz="0 0 ${wheel_radius - wheel_axis_z}" />
+    </joint>
     <link name="base_link">
         <visual>
@@ -32,5 +43,5 @@
             <parent link="base_link" />
             <child link="${wheel_name}" />
-            <origin xyz="${reflect_x * (base_length/2 - wheel_radius)} ${reflect_y * half_track} ${lowrider-(base_height/2 - 0.02)}" rpy="1.57 0 0" />
+            <origin xyz="${reflect_x * (base_length/2 - wheel_radius)} ${reflect_y * half_track} ${wheel_axis_z}" rpy="1.57 0 0" />
             <axis xyz="0 0 1" />
         </joint>

Commit message: Kodutöö 3

File: urdf/fourwheeler.urdf.xacro (robot description, xacro)
@@ -2,6 +2,6 @@
 <robot name="fourwheeler" xmlns:xacro="http://www.ros.org/wiki/xacro">
     <!-- constants; original values are in comments -->
-    <xacro:property name="base_width" value="0.32"/> <!-- 0.32 -->
-    <xacro:property name="base_length" value="0.43"/> <!-- 0.43 -->
+    <xacro:property name="base_width" value="1.32"/> <!-- 0.32 -->
+    <xacro:property name="base_length" value="0.8"/> <!-- 0.43 -->
     <xacro:property name="base_height" value="0.14"/> <!-- 0.14 -->
     <xacro:property name="wheel_width" value="0.05"/> <!-- 0.05 -->
